File: IcePi_Zero_PMOD_Breakout.kicad_pcb (KiCad board)
At the start: 4 copper layers, 30 x 88 mm, 40 parts, among them J1 Conn_02x20_Odd_Even, J2 Conn_02x06_Odd_Even, J3 Conn_02x06_Odd_Even, J4 Conn_02x06_Odd_Even, J5 Conn_02x06_Odd_Even, SW1 SW_Push, SW2 SW_Push, SW3 SW_Push, SW4 SW_Push

Commit message: Need to simplify traces to allow for length matching
Other:
- board text added: "Simplify pinout, tell the user to deal with it?"
Changed lines of the file:
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@@
+		)
+	)
+	(gr_text "Simplify pinout, tell the user to deal with it?"
+		(at 119.38 51.308 0)
+		(layer "Cmts.User")
+		(effects
+			(font
+				(size 1 1)
+				(thickness 0.15)
+			)
+			(justify left bottom)
 		)
 	)
